File: encoder.kicad_pcb (KiCad board)
At the start: 2 copper layers, 22 x 23.9 mm, 15 parts, among them P1 Molex PicoBlade 6 Right, U1 TLE5012B

Commit message: Add version text.
Other:
- board text added: "V.2023.0.2"
Changed lines of the file:
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@@
   (gr_line (start 145.2511 108.87703) (end 151.7511 108.87703)
     (stroke (width 0.0127) (type solid)) (layer "User.1"))
+  (gr_text "V.2023.0.2" (at 151.96175 104.92352) (layer "B.SilkS")
+    (effects (font (size 1.5 1.5) (thickness 0.3) bold) (justify left bottom mirror))
+  )
   (segment (start 149.08675 98.32352) (end 149.08675 96.84852) (width 0.5) (layer "F.Cu") (net 1))
   (segment (start 147.84375 101.06152) (end 147.84375 100.11052) (width 0.5) (layer "F.Cu") (net 1))
